Commit message: Initial commit for sim with amcl and move_base

File: nexus_4wd_mecanum_description/urdf/nexus_4wd_mecanum.xacro (robot description, xacro)
@@ -326,15 +326,54 @@
     </visual>
   </link>
+  <joint name="top_sensor_joint" type="fixed">
+    <origin xyz="0.0 0 0.10" rpy="0 0 0" />
+    <parent link="base_link"/>
+    <child link="top_sensor" />
+  </joint>
+  <link name="top_sensor">
+    <visual>
+      <origin xyz="0 0 0" rpy="0 0 0" />
+      <geometry>
+        <!--<mesh filename="package://nexus_4wd_mecanum_description/meshes/urm04.STL" scale="0.001 0.001 0.001"/>-->
+        <cylinder radius="${wheel_radius}" length="${wheel_width}"/>
+      </geometry>
+      <material name="black" />
+    </visual>
+  </link>
+  <!-- <joint name="bumper_joint" type="fixed">
+    <origin xyz="0.0 0 0.0" rpy="0 0 0" />
+    <parent link="base_link"/>
+    <child link="bumper_link" />
+  </joint>
+  <link name="bumper_link">
+    <collision>
+      <origin xyz="0 0 0" rpy="0 0 0" />
+      <geometry>
+        <box radius="${wheel_radius}" length="${wheel_width}"/>
+      </geometry>
+    </collision>
+  </link> -->
   <!-- Include controller plugin for Gazebo -->
   <xacro:include filename="$(find nexus_4wd_mecanum_description)/urdf/nexus_4wd_mecanum.gazebo" />
   <!-- Include URM04 ultrasonic range finders -->
   <xacro:include filename="$(find nexus_4wd_mecanum_description)/urdf/urm04_sensor.xacro"/>
+  <xacro:include filename="$(find nexus_4wd_mecanum_description)/urdf/lidar_sensor.xacro"/>
   <!-- front sensor -->
-  <xacro:urm04_sensor frame_name="front_sensor" ros_topic="front_sensor" update_rate="10" min_range="0.04" max_range="2.5" horizontal_field_of_view="1.04" vertical_field_of_view="0.04" ray_count="2" />
+  <!-- <xacro:urm04_sensor frame_name="front_sensor" ros_topic="front_sensor" update_rate="10" min_range="0.04" max_range="2.5" horizontal_field_of_view="1.04" vertical_field_of_view="0.04" ray_count="2" /> -->
   <!-- left sensor -->
-  <xacro:urm04_sensor frame_name="left_sensor" ros_topic="left_sensor" update_rate="10" min_range="0.04" max_range="2.5" horizontal_field_of_view="1.04" vertical_field_of_view="0.04" ray_count="2" />
+  <!-- <xacro:urm04_sensor frame_name="left_sensor" ros_topic="left_sensor" update_rate="10" min_range="0.04" max_range="2.5" horizontal_field_of_view="1.04" vertical_field_of_view="0.04" ray_count="2" /> -->
   <!-- right sensor -->
-  <xacro:urm04_sensor frame_name="right_sensor" ros_topic="right_sensor" update_rate="10" min_range="0.04" max_range="2.5" horizontal_field_of_view="1.04" vertical_field_of_view="0.04" ray_count="2" />
+  <!-- <xacro:urm04_sensor frame_name="right_sensor" ros_topic="right_sensor" update_rate="10" min_range="0.04" max_range="2.5" horizontal_field_of_view="1.04" vertical_field_of_view="0.04" ray_count="2" /> -->
   <!-- rear sensor -->
-  <xacro:urm04_sensor frame_name="rear_sensor" ros_topic="rear_sensor" update_rate="10" min_range="0.04" max_range="2.5" horizontal_field_of_view="1.04" vertical_field_of_view="0.04" ray_count="2" />
+  <!-- <xacro:urm04_sensor frame_name="rear_sensor" ros_topic="rear_sensor" update_rate="10" min_range="0.04" max_range="2.5" horizontal_field_of_view="1.04" vertical_field_of_view="0.04" ray_count="2" /> -->
+  <xacro:lidar_sensor frame_name="top_sensor" ros_topic="scan" update_rate="30" min_range="0.01" max_range="30" horizontal_field_of_view="6.28" vertical_field_of_view="0.0" ray_count="720" />
+<!--
+  <gazebo reference="">
+  <plugin name="gazebo_ros_bumper_controller" filename="libgazebo_ros_bumper.so">
+    <alwaysOn>true</alwaysOn>
+    <updateRate>30</updateRate>
+    <bumperTopicName>bumper</bumperTopicName>
+    <frameName>map</frameName>
+  </plugin>
+  </gazebo> -->
 </robot>
